File: SCH/BlockDiagram.sch (KiCad schematic (older format))
At the start: 4 parts, among them SW1 SW_DIP_x03

Commit message: Rev2: Register I/O logic, clock design changes, minor fixes
Parts:
- removed SW1: SW_DIP_x03, symbol Switch:SW_DIP_x03
- added R7: 10K, symbol Device:R
- added SW1: SW_DIP_x04, symbol Switch:SW_DIP_x04
Connections:
- wire segments 21 -> 34
Other:
- moved on the sheet: R1, R2, R3
Changed lines of the file:
@@
 $Descr A3 16535 11693
 encoding utf-8
-Sheet 2 3
-Title "Hierarchy"
+Sheet 2 11
+Title "REGISTER_FILE"
 Date ""
-Rev ""
+Rev "1"
 Comp "IEEE Student Branch 1019"
 Comment1 ""
@@
 $EndDescr
 $Sheet
-S 8000 5800 900  600
+S 5550 5300 900  600
 U 618C425E
 F0 "CLK" 50
 F1 "ClockCtrl.sch" 50
-F2 "CLK" O R 8900 5950 50
-F3 "!CLK" O R 8900 6200 50
-F4 "CLK_SEL" I L 8000 6050 50
+F2 "CLK" O R 6450 5450 50
+F3 "!CLK" O R 6450 5700 50
+F4 "~HLT" I L 5550 5700 50
+F5 "CLK_SEL[2..0]" I L 5550 5450 50
 $EndSheet
-Text Label 7200 6050 0    50   ~ 0
+Text Label 4750 5450 0    50   ~ 0
 CLKSEL[0..2]
 $Comp
 L power:GND #PWR01
 U 1 1 61969A00
-P 6000 6100
-F 0 "#PWR01" H 6000 5850 50  0001 C CNN
-F 1 "GND" H 6005 5927 50  0000 C CNN
-F 2 "" H 6000 6100 50  0001 C CNN
-F 3 "" H 6000 6100 50  0001 C CNN
-	1    6000 6100
+P 3550 5500
+F 0 "#PWR01" H 3550 5250 50  0001 C CNN
+F 1 "GND" H 3555 5327 50  0000 C CNN
+F 2 "" H 3550 5500 50  0001 C CNN
+F 3 "" H 3550 5500 50  0001 C CNN
+	1    3550 5500
 	1    0    0    -1
 $EndComp
@@
 L Device:R R1
 U 1 1 6196A13F
-P 6250 4900
-F 0 "R1" V 6043 4900 50  0000 C CNN
-F 1 "10K" V 6134 4900 50  0000 C CNN
-F 2 "" V 6180 4900 50  0001 C CNN
-F 3 "~" H 6250 4900 50  0001 C CNN
-	1    6250 4900
+P 3800 4300
+F 0 "R1" V 3593 4300 50  0000 C CNN
+F 1 "10K" V 3684 4300 50  0000 C CNN
+F 2 "" V 3730 4300 50  0001 C CNN
+F 3 "~" H 3800 4300 50  0001 C CNN
+	1    3800 4300
 	0    1    1    0
 $EndComp
@@
 L Device:R R2
 U 1 1 6196A94E
-P 6250 5200
-F 0 "R2" V 6043 5200 50  0000 C CNN
-F 1 "10K" V 6134 5200 50  0000 C CNN
-F 2 "" V 6180 5200 50  0001 C CNN
-F 3 "~" H 6250 5200 50  0001 C CNN
-	1    6250 5200
+P 3800 4600
+F 0 "R2" V 3593 4600 50  0000 C CNN
+F 1 "10K" V 3684 4600 50  0000 C CNN
+F 2 "" V 3730 4600 50  0001 C CNN
+F 3 "~" H 3800 4600 50  0001 C CNN
+	1    3800 4600
 	0    1    1    0
 $EndComp
@@
 L Device:R R3
 U 1 1 6196ABB8
-P 6250 5500
-F 0 "R3" V 6043 5500 50  0000 C CNN
-F 1 "10K" V 6134 5500 50  0000 C CNN
-F 2 "" V 6180 5500 50  0001 C CNN
-F 3 "~" H 6250 5500 50  0001 C CNN
-	1    6250 5500
-	0    1    1    0
-$EndComp
-Wire Wire Line
-	6000 4900 6100 4900
-Wire Wire Line
-	6000 5200 6100 5200
-Connection ~ 6000 5200
-Wire Wire Line
-	6000 5200 6000 4900
-Wire Wire Line
-	6100 5500 6000 5500
-Connection ~ 6000 5500
-Wire Wire Line
-	6000 5500 6000 5200
-$Comp
-L Switch:SW_DIP_x03 SW1
-U 1 1 6196C00A
-P 6800 4500
-F 0 "SW1" V 6754 4830 50  0000 L CNN
-F 1 "SW_DIP_x03" V 6845 4830 50  0000 L CNN
-F 2 "" H 6800 4500 50  0001 C CNN
-F 3 "~" H 6800 4500 50  0001 C CNN
-	1    6800 4500
-	0    1    1    0
-$EndComp
+P 3800 4900
+F 0 "R3" V 3593 4900 50  0000 C CNN
+F 1 "10K" V 3684 4900 50  0000 C CNN
+F 2 "" V 3730 4900 50  0001 C CNN
+F 3 "~" H 3800 4900 50  0001 C CNN
+	1    3800 4900
+	0    1    1    0
+$EndComp
+Wire Wire Line
+	3550 4300 3650 4300
+Wire Wire Line
+	3550 4600 3650 4600
+Connection ~ 3550 4600
+Wire Wire Line
+	3550 4600 3550 4300
+Wire Wire Line
+	3650 4900 3550 4900
+Connection ~ 3550 4900
+Wire Wire Line
+	3550 4900 3550 4600
 $Comp
 L power:VCC #PWR02
 U 1 1 6196E08C
-P 6900 3900
-F 0 "#PWR02" H 6900 3750 50  0001 C CNN
-F 1 "VCC" H 6915 4073 50  0000 C CNN
-F 2 "" H 6900 3900 50  0001 C CNN
-F 3 "" H 6900 3900 50  0001 C CNN
-	1    6900 3900
+P 4450 3300
+F 0 "#PWR02" H 4450 3150 50  0001 C CNN
+F 1 "VCC" H 4465 3473 50  0000 C CNN
+F 2 "" H 4450 3300 50  0001 C CNN
+F 3 "" H 4450 3300 50  0001 C CNN
+	1    4450 3300
 	1    0    0    -1
 $EndComp
 Wire Wire Line
-	6900 3900 6900 4050
-Wire Wire Line
-	6900 4050 6800 4050
-Wire Wire Line
-	6800 4050 6800 4200
-Wire Wire Line
-	6900 4200 6900 4050
-Connection ~ 6900 4050
-Wire Wire Line
-	6900 4050 7000 4050
-Wire Wire Line
-	7000 4050 7000 4200
+	4450 3300 4450 3450
+Wire Wire Line
+	4450 3450 4350 3450
+Wire Wire Line
+	4350 3450 4350 3600
+Wire Wire Line
+	4450 3600 4450 3450
+Connection ~ 4450 3450
+Wire Wire Line
+	4450 3450 4550 3450
+Wire Wire Line
+	4550 3450 4550 3600
 Entry Wire Line
-	6800 5950 6900 6050
+	4350 5350 4450 5450
 Entry Wire Line
-	6900 5950 7000 6050
+	4450 5350 4550 5450
 Entry Wire Line
-	7000 5950 7100 6050
-Wire Wire Line
-	6400 4900 6800 4900
-Connection ~ 6800 4900
-Wire Wire Line
-	6800 4900 6800 4800
-Wire Wire Line
-	6400 5200 6900 5200
-Connection ~ 6900 5200
-Wire Wire Line
-	6900 5200 6900 4800
-Wire Wire Line
-	7000 4800 7000 5500
-Wire Wire Line
-	6400 5500 7000 5500
-Connection ~ 7000 5500
-Wire Wire Line
-	6800 4900 6800 5950
-Wire Wire Line
-	6900 5200 6900 5950
-Wire Wire Line
-	7000 5500 7000 5950
-Wire Wire Line
-	6000 5500 6000 6100
+	4550 5350 4650 5450
+Wire Wire Line
+	3950 4300 4350 4300
+Connection ~ 4350 4300
+Wire Wire Line
+	4350 4300 4350 4200
+Wire Wire Line
+	3950 4600 4450 4600
+Connection ~ 4450 4600
+Wire Wire Line
+	4450 4600 4450 4200
+Wire Wire Line
+	4550 4200 4550 4900
+Wire Wire Line
+	3950 4900 4550 4900
+Connection ~ 4550 4900
+Wire Wire Line
+	4350 4300 4350 5350
+Wire Wire Line
+	4450 4600 4450 5350
+Wire Wire Line
+	4550 4900 4550 5350
+Wire Wire Line
+	3550 4900 3550 5200
+$Sheet
+S 4250 5850 1000 600
+U 61AF8F76
+F0 "CLK_HLT_CIRCUIT" 50
+F1 "CLK_HLT_CIRCUIT.sch" 50
+F2 "~PC-OVF" I L 4250 6150 50
+F3 "~IO-WAIT" I L 4250 6300 50
+F4 "HLT" I L 4250 6000 50
+F5 "~CLK_HLT" O R 5250 6000 50
+$EndSheet
+Wire Wire Line
+	5250 6000 5400 6000
+Wire Wire Line
+	5400 6000 5400 5700
+Wire Wire Line
+	5400 5700 5550 5700
+$Comp
+L Switch:SW_DIP_x04 SW1
+U 1 1 61B7F96D
+P 4350 3900
+F 0 "SW1" V 4304 4230 50  0000 L CNN
+F 1 "SW_DIP_x04" V 4395 4230 50  0000 L CNN
+F 2 "" H 4350 3900 50  0001 C CNN
+F 3 "~" H 4350 3900 50  0001 C CNN
+	1    4350 3900
+	0    1    1    0
+$EndComp
+Wire Wire Line
+	4250 3600 4250 3450
+Wire Wire Line
+	4250 3450 4350 3450
+Connection ~ 4350 3450
+$Comp
+L Device:R R7
+U 1 1 61B80837
+P 3800 5200
+F 0 "R7" V 3593 5200 50  0000 C CNN
+F 1 "10K" V 3684 5200 50  0000 C CNN
+F 2 "" V 3730 5200 50  0001 C CNN
+F 3 "~" H 3800 5200 50  0001 C CNN
+	1    3800 5200
+	0    1    1    0
+$EndComp
+Wire Wire Line
+	3650 5200 3550 5200
+Connection ~ 3550 5200
+Wire Wire Line
+	3550 5200 3550 5500
+Wire Wire Line
+	3950 5200 4100 5200
+Wire Wire Line
+	4250 5200 4250 4200
+Wire Wire Line
+	4100 5200 4100 6000
+Wire Wire Line
+	4100 6000 4250 6000
+Connection ~ 4100 5200
+Wire Wire Line
+	4100 5200 4250 5200
+$Sheet
+S 7500 4200 1700 1300
+U 6197E548
+F0 "REGISTER_FILE" 50
+F1 "REGISTER_FILE.sch" 50
+F2 "INC" I L 7500 5350 50
+F3 "IN[3..0]" I L 7500 4350 50
+F4 "~RST" I L 7500 5250 50
+F5 "~CLK" I L 7500 5450 50
+F6 "A[3..0]" O R 9200 4350 50
+F7 "B[3..0]" O R 9200 5250 50
+F8 "AUX[7..0]" O R 9200 5400 50
+F9 "IN_SEL[2..0]" I L 7500 4500 50
+F10 "IN_EN" I L 7500 4600 50
+F11 "A_SEL[2..0]" I L 7500 4750 50
+F12 "A_EN" I L 7500 4850 50
+F13 "B_SEL[2..0]" I L 7500 5000 50
+F14 "B_EN" I L 7500 5100 50
+$EndSheet
+Wire Wire Line
+	6450 5450 7500 5450
 Wire Bus Line
-	6650 6050 8000 6050
+	4200 5450 5550 5450
 $EndSCHEMATC

Commit message: Rev3 e ICT
Other:
- moved on the sheet: R1, R2, R3, R7, SW1
