File: SCH/ClockCtrl.sch (KiCad schematic (older format))
At the start: 13 parts, among them SW2 MANUAL_CLK_BTN, U1 74HC14, U2 NE555P, U3 74151

Commit message: Rev2: Register I/O logic, clock design changes, minor fixes
Parts:
- removed U3: 74151, symbol 74xx_IEEE:74151
- added C11, C8: 100n, symbol Device:C
- added C7: 10n, symbol Device:C
- added D1: 1N4148, Diode_THT:D_DO-35_SOD27_P7.62mm_Horizontal, symbol Diode:1N4148
- added D2: MAN_CLK, symbol Device:LED
- added R12, R8: 10k, symbol Device:R
- added R9: 330, symbol Device:R
- added SW3: SW_SPST, symbol Switch:SW_SPST
- added unit 3 of U1
- added U3: 74HC163, symbol 74xx:74LS163
- added U4: 74HC14, symbol 74xx:74HC14
- added U5: 74HC151, symbol 74xx:74LS151
- added U8: 74HC157, symbol 74xx:74LS157
- R5: value 100k -> 1M
Connections:
- net labels added: CLKSEL[2..0], CLK_100, CLK_12Hz5, CLK_25, CLK_3Hz125, CLK_50, CLK_6Hz25, CLK_SEL[2..0], ~CLK, ~CLK_MAN, ~HLT
- net labels removed: !CLK, CLKSEL[0..2], CLK_1KHz, CLK_SEL
- wire segments 71 -> 137
Other:
- note added: "A regime la tensione sul pin 2 è uguale a VCC, mentre\nla tensione ai capi del condensatore è nulla.\nAlla pressione di SW2 la tensione ai capi del condensatore\ndiviene VCC, di conseguenza quest'ultimo inizia a caricarsi,\n portando la tensione sul pin 2 di U2 a 0V per poi \ncrescere secondo la legge V(t) = VCC(1 - e^(-t/RC)), RC = 100u\nSe SW2 viene rilasciato, la tensione ai capi del condensat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"
- note added: "Notare che l'output TC non è\nun clock con DC 50% ma è solo \nun impulso limitato.\nDa verificare il corretto \nfunzionamento del sistema con \nun clock così veloce"
- moved on the sheet: C1, C2, C3, C4, C5, R4, R5, R6, SW2, U1A, U1B, U2
