File: SCH/TeToLogic.sch (KiCad schematic (older format))
At the start: 0 parts

Commit message: Rev2: Register I/O logic, clock design changes, minor fixes
Other:
- note added: "1"
- note added: "2"
- note added: "24/11"
- note added: "29/11"
- note added: "Aggiunta contatore per divisore frequenza. modifica input pushbutton in CLK_GEN. Creazione circuito HLT, Aggiunta bit a CLK_SELECT. Aggiunta registri"
- note added: "Fix convenzione dei nomi, register selection and I/O logic"
Changed lines of the file:
@@
 $Descr A3 16535 11693
 encoding utf-8
-Sheet 1 3
-Title "TeToLogic"
+Sheet 1 11
+Title "REGISTER_FILE"
 Date "2021-11-10"
 Rev ""
-Comp "IEEE Sudent Branch 1019"
+Comp "IEEE Student Branch 1019"
 Comment1 ""
 Comment2 ""
@@
 Text Notes 1000 3200 0    315  Italic 0
 IEEE Student Branch 1019, University of Brescia
-Wire Notes Line
-	950  3650 15800 3650
-Wire Notes Line
-	950  4000 15800 4000
-Text Notes 950  3900 0    157  ~ 0
+Text Notes 1100 3900 0    71   ~ 0
 Rev.
-Text Notes 1750 3900 0    157  ~ 0
+Text Notes 1750 3900 0    71   ~ 0
 Date
-Text Notes 2700 3900 0    157  ~ 0
+Text Notes 2700 3900 0    71   ~ 0
 Revision Description
-Wire Notes Line
-	1600 3650 1600 10000
-Wire Notes Line
-	2650 3650 2650 10000
-Text Notes 1100 4250 0    157  ~ 0
-0
-Text Notes 1750 4250 0    157  ~ 0
+Text Notes 1750 4100 0    59   ~ 0
 10/11
-Text Notes 2850 4250 0    157  ~ 0
+Text Notes 2700 4100 0    59   ~ 0
 Creazione progetto, Prima progettazione del generatore di clock e clk multiplexer
-Wire Notes Line
-	950  4300 15800 4300
 $Sheet
 S 16700 11300 800  200
@@
 F1 "BlockDiagram.sch" 157
 $EndSheet
+Text Notes 1100 4300 0    59   ~ 0
+1
+Text Notes 2700 4300 0    59   ~ 0
+Aggiunta contatore per divisore frequenza. modifica input pushbutton in CLK_GEN. Creazione circuito HLT, Aggiunta bit a CLK_SELECT. Aggiunta registri
+Text Notes 1100 4100 0    59   ~ 0
+0
+Wire Notes Line
+	15900 3950 1000 3950
+Wire Notes Line
+	1000 4150 15900 4150
+Text Notes 1750 4300 0    59   ~ 0
+24/11
+Text Notes 2700 4500 0    59   ~ 0
+Fix convenzione dei nomi, register selection and I/O logic
+Wire Notes Line
+	1000 4350 15900 4350
+Text Notes 1100 4500 0    59   ~ 0
+2
+Text Notes 1750 4500 0    59   ~ 0
+29/11
 $EndSCHEMATC

Commit message: Rev3 e ICT
Other:
- note added: "15/12"
- note added: "3"
- note added: "Alu e interconnessione con i registri. Logo nel cartiglio e fix minori"
Changed lines of the file:
@@
 $Descr A3 16535 11693
 encoding utf-8
-Sheet 1 11
-Title "REGISTER_FILE"
+Sheet 1 13
+Title ""
 Date "2021-11-10"
 Rev ""
@@
 Text Notes 1750 4500 0    59   ~ 0
 29/11
+Text Notes 2700 4700 0    59   ~ 0
+Alu e interconnessione con i registri. Logo nel cartiglio e fix minori
+Wire Notes Line
+	1000 4550 15900 4550
+Text Notes 1100 4700 0    59   ~ 0
+3
+Text Notes 1750 4700 0    59   ~ 0
+15/12
 $EndSCHEMATC
